Commit message: 修改模型
就该模型参数，现在设定的误差参数和matlab中计算的结果一致了。

File: set_up_tf/urdf/my_robot.xacro (robot description, xacro)
@@ -4,15 +4,15 @@
 	<xacro:property name="dgree" value="${PI/180}" />
 	<xacro:property name="MM" value="0.001" />
-	<xacro:property name="D_th1" value="${0.2*dgree}" />
-	<xacro:property name="D_th2" value="${0.3*dgree}" />
-	<xacro:property name="D_th3" value="${0.4*dgree}" />
-	<xacro:property name="D_th4" value="${0.5*dgree}" />
-	<xacro:property name="D_th5" value="${0.6*dgree}" />
-	<xacro:property name="D_th6" value="${0.7*dgree}" />
-	<xacro:property name="D_L1" value="${0.1*MM}" />
-	<xacro:property name="D_L2" value="${0.2*MM}" />
-	<xacro:property name="D_L3" value="${0.3*MM}" />
-	<xacro:property name="D_L4" value="${0.4*MM}" />
-	<xacro:property name="D_L5" value="${0.5*MM}" />
+	<xacro:property name="D_th1" value="${0.1*dgree}" />
+	<xacro:property name="D_th2" value="${0.2*dgree}" />
+	<xacro:property name="D_th3" value="${0.3*dgree}" />
+	<xacro:property name="D_th4" value="${0.4*dgree}" />
+	<xacro:property name="D_th5" value="${0.5*dgree}" />
+	<xacro:property name="D_th6" value="${0.6*dgree}" />
+	<xacro:property name="D_L1" value="${0.0*MM}" />
+	<xacro:property name="D_L2" value="${0.0*MM}" />
+	<xacro:property name="D_L3" value="${0.0*MM}" />
+	<xacro:property name="D_L4" value="${0.0*MM}" />
+	<xacro:property name="D_L5" value="${0.0*MM}" />
 	<link name="base_link">
 		<visual>
@@ -99,5 +99,5 @@
 		<child link="link_2"/>
 		<limit effort="100" velocity="180" lower="-3.14" upper="3.14"/>
-		<origin xyz="${0.1+D_L1} 0 0" rpy="-1.57 0 ${D_th2}"/>
+		<origin xyz="${0.1+D_L1} 0 0" rpy="${-PI/2} ${D_th2} 0"/>
 		<axis xyz="0 0 1"/>
 	</joint>
@@ -106,5 +106,5 @@
 		<child link="link_3"/>
 		<limit effort="100" velocity="180" lower="-3.14" upper="3.14"/>
-		<origin xyz="0 ${-0.3+D_L2} 0" rpy="3.14 0 ${-1.57+D_th3}"/>
+		<origin xyz="0 ${-0.3-D_L2} 0" rpy="${PI} 0 ${-PI/2-D_th3}"/>
 		<axis xyz="0 0 1"/>
 	</joint>
@@ -113,5 +113,5 @@
 		<child link="link_4"/>
 		<limit effort="100" velocity="180" lower="-3.14" upper="3.14"/>
-		<origin xyz="${0.02+D_L3} 0 0" rpy="-1.57 0 ${D_th4}"/>
+		<origin xyz="${0.02+D_L3} 0 0" rpy="${-PI/2} ${D_th4} 0"/>
 		<axis xyz="0 0 1"/>
 	</joint>
@@ -120,5 +120,5 @@
 		<child link="link_5"/>
 		<limit effort="100" velocity="180" lower="-3.14" upper="3.14"/>
-		<origin xyz="0 0 ${-0.3+D_L4}" rpy="1.57 0 ${D_th5}"/>
+		<origin xyz="0 0 ${-0.3+D_L4}" rpy="${PI/2} -${D_th5} 0"/>
 		<axis xyz="0 0 1"/>
 	</joint>
@@ -127,5 +127,5 @@
 		<child link="link_6"/>
 		<limit effort="100" velocity="180" lower="-3.14" upper="3.14"/>
-		<origin xyz="0 ${-0.1+D_L5} 0" rpy="1.57 0 ${D_th6}"/>
+		<origin xyz="0 ${-0.1+D_L5} 0" rpy="${PI/2} -${D_th6} 0"/>
 		<axis xyz="0 0 1"/>
 	</joint>
