Commit message: 将controller放到这个包下编译生成

File: set_up_tf/urdf/my_robot.urdf (robot description, URDF)
Before this commit: robot myFirst, 7 links, 7 joints
Joints:
- joint joint_1: origin xyz=0 0 0.1 rpy=0 0 0 -> xyz=0 0 0.1 rpy=0 0 0.00174532922222
- joint joint_2: origin xyz=0.1 0 0 rpy=-1.57 0 0 -> xyz=0.1001 0 0 rpy=-1.5707963 0.00349065844444 0
- joint joint_3: origin xyz=0 -0.3 0 rpy=3.14 0 -1.57 -> xyz=0 -0.3002 0 rpy=3.1415926 0 -1.57603228767
- joint joint_4: origin xyz=0.02 0 0 rpy=-1.57 0 0 -> xyz=0.0203 0 0 rpy=-1.5707963 0.00698131688889 0
- joint joint_5: origin xyz=0 0 -0.3 rpy=1.57 0 0 -> xyz=0 0 -0.2996 rpy=1.5707963 -0.00872664611111 0
- joint joint_6: origin xyz=0 -0.1 0 rpy=1.57 0 0 -> xyz=0 -0.0995 0 rpy=1.5707963 -0.0104719753333 0
